Commit message: Added Rviz Visualization Node

File: crazyflie_description/urdf/crazyflie.urdf.xacro (robot description, xacro)
@@ -8,4 +8,10 @@
       <inertia ixx="0.01152" ixy="0.0" ixz="0.0" iyy="0.01152" iyz="0.0" izz="0.0218" />
     </inertial>
+    <joint name="crazyflie_joint" type="fixed">
+      <origin xyz="0 0 0"
+        rpy="0 0 0"/>
+      <parent link="world"/>
+      <child link="base_link"/>
+  </joint>
     <visual>
       <origin xyz="0 0 0" rpy="0 0 0" />

File: crazyflie_description/urdf/crazyflie2.urdf.xacro (robot description, xacro)
@@ -3,4 +3,12 @@
   <xacro:property name="rotor_drag_coefficient" value="1.8580e-05"/> <!-- [N.m.s^2] -->
   <xacro:property name="moment_constant" value="0.005"/> <!-- [N.s^2] -->
+  <xacro:property name="obj_pose_file" value="$(find maps)/config/cylinder_gen.yaml"/>
+  <xacro:property name="obj_pose" value="${xacro.load_yaml(obj_pose_file)}"/>
+  <xacro:property name="x1" value="${obj_pose['obstacles'][0]['x']}" />
+  <xacro:property name="y1" value="${obj_pose['obstacles'][0]['y']}" />
+  <xacro:property name="r1" value="${obj_pose['obstacles'][0]['r']}" />
+  <xacro:property name="x2" value="${obj_pose['obstacles'][1]['x']}" />
+  <xacro:property name="y2" value="${obj_pose['obstacles'][1]['y']}" />
+  <xacro:property name="r2" value="${obj_pose['obstacles'][1]['r']}" />
   <link name="base_link">
     <inertial>
